File: M68K-BREAKOUT.sch (KiCad schematic (older format))
At the start: 27 parts, among them U1 68010D, U2 74ALVC164245, U3 74ALVC164245, U4 74ALVC164245, U5 74ALVC164245, U6 74LVC06

Commit message: complete electrical layout for the silicon centipede charmer
Parts:
- removed C12, C13, C14, C15, C16, C17, C18, C19: 100nF, Capacitor_SMD:C_0603_1608Metric_Pad1.08x0.95mm_HandSolder, symbol Device:C_Small
- added J1: Data, Connector_PinHeader_2.00mm:PinHeader_2x09_P2.00mm_Vertical, symbol Connector_Generic:Conn_02x09_Odd_Even
- added J2: Bus Signals, Connector_PinHeader_2.00mm:PinHeader_2x09_P2.00mm_Vertical, symbol Connector_Generic:Conn_02x09_Odd_Even
- added J3: Address, Connector_PinHeader_2.00mm:PinHeader_2x09_P2.00mm_Vertical, symbol Connector_Generic:Conn_02x09_Odd_Even
- added J4: Function Code and Lower Address, Connector_PinHeader_2.00mm:PinHeader_2x09_P2.00mm_Vertical, symbol Connector_Generic:Conn_02x09_Odd_Even
- added R3: 2.2K, Resistor_SMD:R_0603_1608Metric_Pad0.98x0.95mm_HandSolder, symbol Device:R_Small_US
Connections:
- net +3V3: now also C10.1, C7.1, C8.1, C9.1, J2.9 (Pin_9), J4.9 (Pin_9)
- net +5V: now also J1.9 (Pin_9), J3.9 (Pin_9), R3.1; no longer C10.1, C7.1, C8.1, C9.1, U1.21 (VPA)
- net GND: now also J1.10 (Pin_10), J2.10 (Pin_10), J3.10 (Pin_10), J4.10 (Pin_10), J4.11 (Pin_11), J4.5 (Pin_5), J4.6 (Pin_6), J4.7 (Pin_7), J4.8 (Pin_8); no longer U4.36 (2A0), U5.36 (2A0), U5.37 (1A7), U5.38 (1A6), U5.40 (1A5), U5.41 (1A4), U5.43 (1A3), U6.10, U6.12, U6.6, U6.8
- net L_FC0: now also J4.3 (Pin_3)
- net L_FC1: now also J4.2 (Pin_2)
- net L_FC2: now also J4.1 (Pin_1)
- net AA8: now reaches U3.26 (2A7)
- net AA8: now also J3.18 (Pin_18)
- net AA9: now reaches U3.27 (2A6)
- net AA9: now also J3.17 (Pin_17)
- net AA10: now reaches U3.29 (2A5)
- net AA10: now also J3.16 (Pin_16)
- net AA11: now reaches U3.30 (2A4)
- net AA11: now also J3.15 (Pin_15)
- net AA12: now reaches U3.32 (2A3)
- net AA12: now also J3.14 (Pin_14)
- net AA13: now reaches U3.33 (2A2)
- net AA13: now also J3.13 (Pin_13)
- net AA14: now reaches U3.35 (2A1)
- net AA14: now also J3.12 (Pin_12)
- net AA15: now reaches U3.36 (2A0)
- net AA15: now also J3.11 (Pin_11)
- net AA16: now reaches U3.37 (1A7)
- net AA16: now also J3.8 (Pin_8)
- net AA17: now reaches U3.38 (1A6)
- net AA17: now also J3.7 (Pin_7)
- net AA18: now reaches U3.40 (1A5)
- net AA18: now also J3.6 (Pin_6)
- net AA19: now reaches U3.41 (1A4)
- net AA19: now also J3.5 (Pin_5)
- net AA20: now reaches U3.43 (1A3)
- net AA20: now also J3.4 (Pin_4)
- net AA21: now reaches U3.44 (1A2)
- net AA21: now also J3.3 (Pin_3)
- net AA22: now reaches U3.46 (1A1)
- net AA22: now also J3.2 (Pin_2)
- net AA23: now reaches U3.47 (1A0)
- net AA23: now also J3.1 (Pin_1)
- net ~L_AS: now reaches U4.26 (2A7)
- net ~L_AS: now also J2.1 (Pin_1)
- net ~L_UDS: now reaches U4.27 (2A6)
- net ~L_UDS: now also J2.2 (Pin_2)
- net ~L_LDS: now reaches U4.29 (2A5)
- net ~L_LDS: now also J2.3 (Pin_3)
- net L_R~W: now reaches U4.30 (2A4)
- net L_R~W: now also J2.4 (Pin_4)
- net ~L_BG: now reaches U4.32 (2A3)
- net ~L_BG: now also J2.5 (Pin_5)
- net ~L_HALT: now reaches U4.33 (2A2)
- net ~L_HALT: now also J2.6 (Pin_6)
- net ~L_RESET: now reaches U4.35 (2A1)
- net ~L_RESET: now also J2.7 (Pin_7)
- net ~L_DTACK: now reaches U4.37 (1A7)
- net ~L_DTACK: now also J2.11 (Pin_11)
- net ~L_BGACK: now reaches U4.38 (1A6)
- net ~L_BGACK: now also J2.12 (Pin_12)
- net ~L_BR: now reaches U4.40 (1A5)
- net ~L_BR: now also J2.13 (Pin_13)
- net L_CLK: now reaches U4.41 (1A4)
- net L_CLK: now also J2.14 (Pin_14)
- net ~L_BERR: now reaches U4.43 (1A3)
- net ~L_BERR: now also J2.15 (Pin_15)
- net ~L_IPL2: now reaches U4.44 (1A2)
- net ~L_IPL2: now also J2.16 (Pin_16)
- net ~L_IPL1: now reaches U4.46 (1A1)
- net ~L_IPL1: now also J2.17 (Pin_17)
- net ~L_IPL0: now reaches U4.47 (1A0)
- net ~L_IPL0: now also J2.18 (Pin_18)
- net DD15: now reaches U2.26 (2A7)
- net DD15: now also J1.18 (Pin_18)
- net DD14: now reaches U2.27 (2A6)
- net DD14: now also J1.17 (Pin_17)
- net DD13: now reaches U2.29 (2A5)
- net DD13: now also J1.16 (Pin_16)
- net DD12: now reaches U2.30 (2A4)
- net DD12: now also J1.15 (Pin_15)
- net DD11: now reaches U2.32 (2A3)
- net DD11: now also J1.14 (Pin_14)
- net DD10: now reaches U2.33 (2A2)
- net DD10: now also J1.13 (Pin_13)
- net DD9: now reaches U2.35 (2A1)
- net DD9: now also J1.12 (Pin_12)
- net DD8: now reaches U2.36 (2A0)
- net DD8: now also J1.11 (Pin_11)
- net DD0: now reaches U2.37 (1A7)
- net DD0: now also J1.8 (Pin_8)
- net DD1: now reaches U2.38 (1A6)
- net DD1: now also J1.7 (Pin_7)
- net DD7: now reaches U2.40 (1A5)
- net DD7: now also J1.6 (Pin_6)
- net DD2: now reaches U2.41 (1A4)
- net DD2: now also J1.5 (Pin_5)
- net DD6: now reaches U2.43 (1A3)
- net DD6: now also J1.4 (Pin_4)
- net DD3: now reaches U2.44 (1A2)
- net DD3: now also J1.3 (Pin_3)
- net DD5: now reaches U2.46 (1A1)
- net DD5: now also J1.2 (Pin_2)
- net DD4: now reaches U2.47 (1A0)
- net DD4: now also J1.1 (Pin_1)
- net LA1 renamed AA1
- net AA1: now also J4.12 (Pin_12)
- net LA2 renamed AA2
- net AA2: now also J4.14 (Pin_14)
- net LA3 renamed AA3
- net AA3: now also J4.16 (Pin_16)
- net LA4 renamed AA4
- net AA4: now also J4.18 (Pin_18)
- net LA5 renamed AA5
- net AA5: now also J4.17 (Pin_17)
- net LA6 renamed AA6
- net AA6: now also J4.15 (Pin_15)
- net LA7 renamed AA7
- net AA7: now also J4.13 (Pin_13)
- net ~HALT_IN renamed HALT_IN
- net HALT_IN: now also J2.8 (Pin_8)
- net ~RESET_IN renamed RESET_IN
- net RESET_IN: now also J4.4 (Pin_4)
- new net: R3.2, U1.21 (VPA)
- no-connect marks 2 -> 13
Other:
- moved on the sheet: C11, U2, U3, U4, U5
