File: M68K-BUS-VOLTAGE-CONVERTER.sch (KiCad schematic (older format))
At the start: 24 parts, among them J1 Data, J2 Bus Signals, J3 Address, J4 Function Code and Lower Addre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, U1 68010D, U2 74ALVC164245, U3 74ALVC164245, U4 74ALVC164245, U5 74ALVC164245, U6 74LVC06

Commit message: Added Bill-of-Materials
Parts:
- C1, C10, C11, C2, C3, C4, C5, C6, C7, C8, C9: Mouser_Link (none) -> https://www.mouser.com/ProductDetail/810-C1608X7R1E104K; Mouser_PN (none) -> 810-C1608X7R1E104K
- R1, R2, R3: Mouser_Link (none) -> https://www.mouser.com/ProductDetail/Bourns/CR0603-FX-2201E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; Mouser_PN (none) -> 652-CR0603FX-2201ELF
- U1: Mouser_Link (none) -> https://www.mouser.com/ProductDetail/575-193964; Mouser_PN (none) -> 575-193964
- U2, U3, U4, U5: Mouser_Link (none) -> https://www.mouser.com/ProductDetail/771-74ALVC164245; Mouser_PN (none) -> 771-74ALVC164245
- U6: Mouser_Link (none) -> https://www.mouser.com/ProductDetail/595-SN74LVC06AD; Mouser_PN (none) -> 595-SN74LVC06AD
